File: hardware/DSP PAW add-on board.kicad_pcb (KiCad board)
At the start: 2 copper layers, 63 x 53.5 mm, 75 parts, among them J1 AudioJack2_Ground, J3 Conn_01x02, J4 Conn_02x03_Odd_Even, J5 AudioJack2_Ground, J7 AudioJack2_Ground, J8 USB_B_Micro, U1 TLV9162, U2 OPA1678, U3 MAX6106, U4 LM27761

Commit message: pcb design finalization
Parts:
- D7: footprint LED_SMD:LED_Kingbright_AAA3528ESGCT -> LED_SMD:LED_LiteOn_LTST-C19HE1WT
- J1, J5, J7: footprint Connector_Audio:Jack_3.5mm_CUI_SJ-3523-SMT_Horizontal -> Connector_Audio:Jack_3.5mm_PJ320D_Horizontal
- moved D1 13.3 mm to (155.0, 115.0)
- moved D2 12.8 mm to (140.5, 115.0)
- moved D3 12.3 mm to (126.0, 115.0)
- moved R26 6.68 mm to (138.5, 115.0), turned to 90 degrees
- moved J4 1.58 mm to (149.2, 105.0)
- moved J7 1.26 mm to (132.2, 118.5), turned to 90 degrees
- moved J5 0.81 mm to (146.8, 118.5), turned to 90 degrees
- moved C8 0.75 mm to (147.0, 96.7)
- moved R23 0.50 mm to (154.6, 81.0)
- moved R25 0.50 mm to (156.2, 81.0)
- moved J1 0.45 mm to (161.2, 118.5), turned to 90 degrees
Routing:
- net SIGNAL_IN: track 21.1 -> 29.5 mm
- net GENERATOR: track 31.0 -> 24.1 mm
- net VCC: track 45.1 -> 46.1 mm
- net Net-(D7-GK): track 2.03 -> 2.86 mm
- net SIGNAL_OUT: track 27.7 -> 27.1 mm
- net PC12/LED_B: track 21.7 -> 22.2 mm
- net PC10/LED_R: track 25.0 -> 25.5 mm
