File: hardware/DSP PAW add-on board.kicad_sch (KiCad schematic)
At the start: 0 parts

Commit message: pcb design finalization
Other:
- note added: "Bill of Materials notes: Manufacturer part numbers were chosen first, and are preferred. LCSC part numbers contain many substitutions that were chosen to match the original components as best as possible: - Capacitor choices are X5R or X7R, +/- 10% tolerance or better, and rated 16V or higher. - MAX6106 reference replaced with REF3020. - TLV9162 replaced with LM833 (used in previous design iterat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"
Changed lines of the file:
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@@
   (title_block
     (title "DSP PAW add-on board")
-    (date "2023-08-15")
+    (date "2023-08-18")
     (company "bitgloo")
     (comment 1 "Released under the CERN Open Hardware Licence Version 2 - Strongly Reciprocal")
   )
+  (text "Bill of Materials notes:\n\nManufacturer part numbers were chosen first, and are preferred. LCSC part numbers\ncontain many substitutions that were chosen to match the original components as\nbest as possible:\n\n  - Capacitor choices are X5R or X7R, +/- 10% tolerance or better, and rated 16V\n    or higher.\n  - MAX6106 reference replaced with REF3020.\n  - TLV9162 replaced with LM833 (used in previous design iteration).\n  - 10kOhm potentiometers replaced with 100kOhm versions."
+    (at 161.29 48.26 0)
+    (effects (font (size 1.27 1.27)) (justify left bottom))
+  )
   (sheet (at 25.4 76.2) (size 50.8 12.7) (fields_autoplaced)
