File: hardware/user_io.kicad_sch (KiCad schematic)
At the start: 6 parts

Commit message: pcb design finalization
Parts:
- D7: LCSC Part # (none) -> C427425; Part Number AAA3528SEEZGKQBKS -> LTST-C19HE1WT
- R17: LCSC Part # (none) -> C23204
- R18, R19: LCSC Part # (none) -> C23350
- RV1, RV2: LCSC Part # (none) -> C330458
Other:
- note added: "Can substitute other resistances given component availability"
- title: User I/O -> DSP PAW add-on board
Changed lines of the file:
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@@
   (paper "A4")
   (title_block
-    (title "User I/O")
-    (date "2023-08-15")
+    (title "DSP PAW add-on board")
+    (date "2023-08-18")
     (company "bitgloo")
     (comment 1 "Released under the CERN Open Hardware Licence Version 2 - Strongly Reciprocal")
@@
   (text "Status LEDs and parameter knobs" (at 115.57 69.85 0)
     (effects (font (size 2.54 2.54) (thickness 0.254) bold) (justify left bottom))
+  )
+  (text "Can substitute other resistances given\ncomponent availability"
+    (at 153.67 124.46 0)
+    (effects (font (size 1.27 1.27)) (justify left bottom))
   )
   (global_label "PC0{slash}POT1" (shape input) (at 153.67 106.68 0) (fields_autoplaced)
@@
       (effects (font (size 1.27 1.27)) hide)
     )
+    (property "DNP" "" (at 193.04 106.68 0)
+      (effects (font (size 1.27 1.27)) hide)
+    )
+    (property "LCSC Part #" "C330458" (at 193.04 106.68 0)
+      (effects (font (size 1.27 1.27)) hide)
+    )
     (pin "1")
     (pin "2")
@@
       (effects (font (size 1.27 1.27)) hide)
     )
+    (property "DNP" "" (at 92.71 106.68 0)
+      (effects (font (size 1.27 1.27)) hide)
+    )
+    (property "LCSC Part #" "C23350" (at 92.71 106.68 0)
+      (effects (font (size 1.27 1.27)) hide)
+    )
     (pin "1")
     (pin "2")
@@
       (effects (font (size 1.27 1.27)) hide)
     )
+    (property "DNP" "" (at 92.71 97.79 0)
+      (effects (font (size 1.27 1.27)) hide)
+    )
+    (property "LCSC Part #" "C23204" (at 92.71 97.79 0)
+      (effects (font (size 1.27 1.27)) hide)
+    )
     (pin "1")
     (pin "2")
@@
       (effects (font (size 1.27 1.27)) hide)
     )
-    (property "Part Number" "AAA3528SEEZGKQBKS" (at 105.41 106.68 0)
+    (property "Part Number" "LTST-C19HE1WT" (at 105.41 106.68 0)
+      (effects (font (size 1.27 1.27)) hide)
+    )
+    (property "DNP" "" (at 105.41 106.68 0)
+      (effects (font (size 1.27 1.27)) hide)
+    )
+    (property "LCSC Part #" "C427425" (at 105.41 106.68 0)
       (effects (font (size 1.27 1.27)) hide)
     )
@@
       (effects (font (size 1.27 1.27)) hide)
     )
+    (property "DNP" "" (at 92.71 115.57 0)
+      (effects (font (size 1.27 1.27)) hide)
+    )
+    (property "LCSC Part #" "C23350" (at 92.71 115.57 0)
+      (effects (font (size 1.27 1.27)) hide)
+    )
     (pin "1")
     (pin "2")
@@
       (effects (font (size 1.27 1.27)) hide)
     )
+    (property "DNP" "" (at 149.86 106.68 0)
+      (effects (font (size 1.27 1.27)) hide)
+    )
+    (property "LCSC Part #" "C330458" (at 149.86 106.68 0)
+      (effects (font (size 1.27 1.27)) hide)
+    )
