File: hardware/analog_io.kicad_sch (KiCad schematic)
At the start: 32 parts, among them U1 TLV9162, U2 OPA1677, U6 OPA1677

Commit message: finalize rev2 schematic
Parts:
- C1: Part Number (none) -> KGM15AR71H151JT
- C4: Part Number (none) -> CC0603KRX7R9BB103
- R1: value 8.45k/0.1% -> 8.45k/1%; Part Number (none) -> CRCW06038K45FKEA
- R12, R13, R17, R18: value 2.49k/0.1% -> 2.49k/0.5%
- R14, R8: value 22.1k/0.1% -> 22.1k/0.5%
- R15, R9: value 6.81k/0.1% -> 6.81k/0.5%
- R2: value 13.2k/0.1% -> 13.3k/1%; Part Number (none) -> RC0603FR-0713K3L
- R28, R29: Part Number (none) -> RC0603JR-07100KL
- R4: Part Number (none) -> RN73R1JTTD1012B25
- R6: Part Number (none) -> RC0603JR-07200RL
- U2, U6: Part Number (none) -> OPA1677DBVR
Changed lines of the file:
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@@
       (effects (font (size 1.27 1.27)) hide)
     )
-    (property "Part Number" "" (at 110.49 54.61 0)
+    (property "Part Number" "RN73R1JTTD1012B25" (at 110.49 54.61 0)
       (effects (font (size 1.27 1.27)) hide)
     )
@@
       (effects (font (size 1.27 1.27)))
     )
-    (property "Value" "2.49k/0.1%" (at 87.63 168.91 90)
+    (property "Value" "2.49k/0.5%" (at 87.63 168.91 90)
       (effects (font (size 1.27 1.27)))
     )
@@
       (effects (font (size 1.27 1.27)))
     )
-    (property "Value" "8.45k/0.1%" (at 52.07 49.53 90)
+    (property "Value" "8.45k/1%" (at 52.07 49.53 90)
       (effects (font (size 1.27 1.27)))
     )
@@
       (effects (font (size 1.27 1.27)) hide)
     )
-    (property "Part Number" "" (at 52.07 52.07 0)
+    (property "Part Number" "CRCW06038K45FKEA" (at 52.07 52.07 0)
       (effects (font (size 1.27 1.27)) hide)
     )
@@
       (effects (font (size 1.27 1.27)))
     )
-    (property "Value" "6.81k/0.1%" (at 128.27 99.06 90)
+    (property "Value" "6.81k/0.5%" (at 128.27 99.06 90)
       (effects (font (size 1.27 1.27)))
     )
@@
       (effects (font (size 1.27 1.27)) hide)
     )
-    (property "Part Number" "" (at 118.745 43.815 0)
+    (property "Part Number" "RN73R1JTTD1012B25" (at 118.745 43.815 0)
       (effects (font (size 1.27 1.27)) hide)
     )
@@
       (effects (font (size 1.27 1.27)))
     )
-    (property "Value" "2.49k/0.1%" (at 88.9 115.57 90)
+    (property "Value" "2.49k/0.5%" (at 88.9 115.57 90)
       (effects (font (size 1.27 1.27)))
     )
@@
       (effects (font (size 1.27 1.27)) hide)
     )
-    (property "Part Number" "" (at 137.16 161.925 0)
+    (property "Part Number" "RC0603JR-07100KL" (at 137.16 161.925 0)
       (effects (font (size 1.27 1.27)) hide)
     )
@@
       (effects (font (size 1.27 1.27)))
     )
-    (property "Value" "13.2k/0.1%" (at 66.04 49.53 90)
+    (property "Value" "13.3k/1%" (at 66.04 49.53 90)
       (effects (font (size 1.27 1.27)))
     )
@@
       (effects (font (size 1.27 1.27)) hide)
     )
-    (property "Part Number" "" (at 66.04 52.07 0)
+    (property "Part Number" "RC0603FR-0713K3L" (at 66.04 52.07 0)
       (effects (font (size 1.27 1.27)) hide)
     )
@@
       (effects (font (size 1.27 1.27)) hide)
     )
+    (property "Part Number" "OPA1677DBVR" (at 87.63 157.48 0)
+      (effects (font (size 1.27 1.27)) hide)
+    )
     (pin "2")
     (pin "5")
@@
       (effects (font (size 1.27 1.27)) hide)
     )
+    (property "Part Number" "OPA1677DBVR" (at 88.9 104.14 0)
+      (effects (font (size 1.27 1.27)) hide)
+    )
     (pin "2")
     (pin "5")
@@
       (effects (font (size 1.27 1.27)))
     )
-    (property "Value" "6.81k/0.1%" (at 127 152.4 90)
+    (property "Value" "6.81k/0.5%" (at 127 152.4 90)
       (effects (font (size 1.27 1.27)))
     )
@@
     )
     (property "DNP" "" (at 163.83 62.23 0)
+      (effects (font (size 1.27 1.27)) hide)
+    )
+    (property "Part Number" "CC0603KRX7R9BB103" (at 163.83 62.23 0)
       (effects (font (size 1.27 1.27)) hide)
     )
@@
       (effects (font (size 1.27 1.27)))
     )
-    (property "Value" "22.1k/0.1%" (at 113.665 99.06 90)
+    (property "Value" "22.1k/0.5%" (at 113.665 99.06 90)
       (effects (font (size 1.27 1.27)))
     )
@@
       (effects (font (size 1.27 1.27)))
     )
-    (property "Value" "22.1k/0.1%" (at 113.03 152.4 90)
+    (property "Value" "22.1k/0.5%" (at 113.03 152.4 90)
       (effects (font (size 1.27 1.27)))
     )
@@
       (effects (font (size 1.27 1.27)) hide)
     )
-    (property "Part Number" "" (at 153.67 54.61 0)
+    (property "Part Number" "RC0603JR-07200RL" (at 153.67 54.61 0)
       (effects (font (size 1.27 1.27)) hide)
     )
@@
       (effects (font (size 1.27 1.27)) hide)
     )
-    (property "Part Number" "" (at 137.16 108.585 0)
+    (property "Part Number" "RC0603JR-07100KL" (at 137.16 108.585 0)
       (effects (font (size 1.27 1.27)) hide)
     )
@@
       (effects (font (size 1.27 1.27)))
     )
-    (property "Value" "2.49k/0.1%" (at 114.3 168.91 90)
+    (property "Value" "2.49k/0.5%" (at 114.3 168.91 90)
       (effects (font (size 1.27 1.27)))
     )
@@
       (effects (font (size 1.27 1.27)) hide)
     )
-    (property "Part Number" "" (at 78.74 43.18 0)
+    (property "Part Number" "KGM15AR71H151JT" (at 78.74 43.18 0)
       (effects (font (size 1.27 1.27)) hide)
     )
@@
       (effects (font (size 1.27 1.27)))
     )
-    (property "Value" "2.49k/0.1%" (at 115.57 115.57 90)
-      (effects (font (size 1.27 1.27)))
-    )
+    (property "Value" "2.49k/0.5%" (at 115.57 115.57 90)
+      (effects (font (size 1.27 1.27)))
+    )
